File: custom65.brd (EAGLE design)
At the start: 100 x 80 mm, 97 parts, among them J1 USB-C-12401598E4#2A, K1 KEYSWITCH-RGBLED-MX-1U-RGB, K10 KEYSWITCH-RGBLED-MX-1U-RGB, K11 KEYSWITCH-RGBLED-MX-1U-RGB, K12 KEYSWITCH-RGBLED-MX-1U-RGB, K13 KEYSWITCH-RGBLED-MX-1U-RGB, K14 KEYSWITCH-RGBLED-MX-1U-RGB, K15 KEYSWITCH-RGBLED-MX-1U-RGB, K16 KEYSWITCH-RGBLED-MX-1U-RGB, K17 KEYSWITCH-RGBLED-MX-1U-RGB, K18 KEYSWITCH-RGBLED-MX-1U-RGB, K19 KEYSWITCH-RGBLED-MX-1U-RGB, K2 KEYSWITCH-RGBLED-MX-1U-RGB, K20 KEYSWITCH-RGBLED-MX-1U-RGB, K21 KEYSWITCH-RGBLED-MX-1U-RGB, K22 KEYSWITCH-RGBLED-MX-1U-RGB, K23 KEYSWITCH-RGBLED-MX-1U-RGB, K24 KEYSWITCH-RGBLED-MX-1U-RGB, K25 KEYSWITCH-RGBLED-MX-1U-RGB, K26 KEYSWITCH-RGBLED-MX-1U-RGB, K27 KEYSWITCH-RGBLED-MX-1U-RGB, K28 KEYSWITCH-RGBLED-MX-1U-RGB, K29 KEYSWITCH-RGBLED-MX-1U-RGB, K3 KEYSWITCH-RGBLED-MX-1U-RGB, K30 KEYSWITCH-RGBLED-MX-1U-RGB, K31 KEYSWITCH-RGBLED-MX-1U-RGB, K32 KEYSWITCH-RGBLED-MX-1U-RGB, K33 KEYSWITCH-RGBLED-MX-1U-RGB, K34 KEYSWITCH-RGBLED-MX-1U-RGB, K35 KEYSWITCH-RGBLED-MX-1U-RGB, K36 KEYSWITCH-RGBLED-MX-1U-RGB, K37 KEYSWITCH-RGBLED-MX-1U-RGB, K38 KEYSWITCH-RGBLED-MX-1U-RGB, K39 KEYSWITCH-RGBLED-MX-1U-RGB, K4 KEYSWITCH-RGBLED-MX-1U-RGB, K40 KEYSWITCH-RGBLED-MX-1U-RGB, K41 KEYSWITCH-RGBLED-MX-1U-RGB, K42 KEYSWITCH-RGBLED-MX-1U-RGB, K5 KEYSWITCH-RGBLED-MX-1U-RGB, K6 KEYSWITCH-RGBLED-MX-1U-RGB, K7 KEYSWITCH-RGBLED-MX-1U-RGB, K8 KEYSWITCH-RGBLED-MX-1U-RGB, K9 KEYSWITCH-RGBLED-MX-1U-RGB

Commit message: updated sch and brd files
Parts:
- removed D15, D16, D17, D18, D19, D20, D21, D22, D23, D24, D25, D26, D28, D29, D30, D31, D32, D33, D34, D35, D36, D37, D38, D39: (no value), Components:DFN0603-2
- removed K17, K18, K19, K20, K21, K22, K23, K24, K25, K26, K27, K28, K29, K30, K31, K32, K33, K34, K35, K36, K37, K38, K39, K40, K41, K42: KEYSWITCH-RGBLED-MX-1U-RGB, Keyboard:MX-1U-RGB
- K1, K10, K11, K12, K13, K14, K15, K16, K2, K3, K4, K5, K6, K7, K8, K9: value KEYSWITCH-RGBLED-MX-1U-RGB -> KEYSWITCH-LEDTHTHOLE-MXHS-1U-LEDTHTHOLE; device Keyboard:MX-1U-RGB -> Keyboard:MXHS-1U-LEDTHTHOLE
- moved K16 547.4 mm to (-378.5, -402.6)
- moved K15 545.5 mm to (-378.5, -387.4)
- moved K14 403.3 mm to (-378.5, -372.1)
- moved K1 402.1 mm to (-378.5, -174.0)
- moved K2 396.0 mm to (-378.5, -189.2)
- moved K13 395.4 mm to (-378.5, -356.9)
- moved K12 388.6 mm to (-378.5, -341.6)
- moved K11 382.9 mm to (-378.5, -326.4)
- moved K3 380.5 mm to (-378.5, -204.5)
- moved K10 378.3 mm to (-378.5, -311.1)
- moved K4 376.5 mm to (-378.5, -219.7)
- moved K9 374.9 mm to (-378.5, -295.9)
- moved K5 373.7 mm to (-378.5, -234.9)
- moved K8 372.8 mm to (-378.5, -280.7)
- moved K6 372.1 mm to (-378.5, -250.2)
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Connections:
- removed net COL10: K11.MX1, K25.MX1, K39.MX1
- removed net COL11: K12.MX1, K26.MX1, K40.MX1
- removed net COL12: K13.MX1, K27.MX1, K41.MX1
- removed net COL13: K14.MX1, K28.MX1, K42.MX1
- removed net COL2: K17.MX1, K3.MX1, K31.MX1
- removed net COL3: K18.MX1, K32.MX1, K4.MX1
- removed net COL4: K19.MX1, K33.MX1, K5.MX1
- removed net COL5: K20.MX1, K34.MX1, K6.MX1
- removed net COL6: K21.MX1, K35.MX1, K7.MX1
- removed net COL7: K22.MX1, K36.MX1, K8.MX1
- removed net COL8: K23.MX1, K37.MX1, K9.MX1
- removed net COL9: K10.MX1, K24.MX1, K38.MX1
- removed net N$19: D14.C, D15.A, K16.MX2
- removed net N$25: D26.C, K28.MX2
- removed net N$26: D25.C, D26.A, K27.MX2
- removed net N$27: D24.C, D25.A, K26.MX2
- removed net N$28: D23.C, D24.A, K25.MX2
- removed net N$29: D22.C, D23.A, K24.MX2
- removed net N$30: D21.C, D22.A, K23.MX2
- removed net N$31: D20.C, D21.A, K22.MX2
- removed net N$32: D19.C, D20.A, K21.MX2
- removed net N$33: D18.C, D19.A, K20.MX2
- removed net N$34: D17.C, D18.A, K19.MX2
- removed net N$35: D16.C, D17.A, K18.MX2
- removed net N$36: D15.C, D16.A, K17.MX2
- removed net N$37: D27.C, D28.A, K30.MX2
- removed net N$38: D39.C, K42.MX2
- removed net N$39: D38.C, D39.A, K41.MX2
- removed net N$40: D37.C, D38.A, K40.MX2
- removed net N$41: D36.C, D37.A, K39.MX2
- removed net N$42: D35.C, D36.A, K38.MX2
- removed net N$43: D34.C, D35.A, K37.MX2
- removed net N$44: D33.C, D34.A, K36.MX2
- removed net N$45: D32.C, D33.A, K35.MX2
- removed net N$46: D31.C, D32.A, K34.MX2
- removed net N$47: D30.C, D31.A, K33.MX2
- removed net N$48: D29.C, D30.A, K32.MX2
- removed net N$49: D28.C, D29.A, K31.MX2
- net COL0: now also K16.MX1; no longer K29.MX1
- net COL1: no longer K16.MX1, K2.MX1, K30.MX1
- net ROW2: now also K16.MX2; no longer K29.MX2
