File: custom65.sch (EAGLE design)
At the start: 97 parts, among them J1 USB-C-12401598E4#2A, K1 KEYSWITCH-RGBLED-MX-1U-RGB, K10 KEYSWITCH-RGBLED-MX-1U-RGB, K11 KEYSWITCH-RGBLED-MX-1U-RGB, K12 KEYSWITCH-RGBLED-MX-1U-RGB, K13 KEYSWITCH-RGBLED-MX-1U-RGB, K14 KEYSWITCH-RGBLED-MX-1U-RGB, K15 KEYSWITCH-RGBLED-MX-1U-RGB, K16 KEYSWITCH-RGBLED-MX-1U-RGB, K17 KEYSWITCH-RGBLED-MX-1U-RGB, K18 KEYSWITCH-RGBLED-MX-1U-RGB, K19 KEYSWITCH-RGBLED-MX-1U-RGB, K2 KEYSWITCH-RGBLED-MX-1U-RGB, K20 KEYSWITCH-RGBLED-MX-1U-RGB, K21 KEYSWITCH-RGBLED-MX-1U-RGB, K22 KEYSWITCH-RGBLED-MX-1U-RGB, K23 KEYSWITCH-RGBLED-MX-1U-RGB, K24 KEYSWITCH-RGBLED-MX-1U-RGB, K25 KEYSWITCH-RGBLED-MX-1U-RGB, K26 KEYSWITCH-RGBLED-MX-1U-RGB, K27 KEYSWITCH-RGBLED-MX-1U-RGB, K28 KEYSWITCH-RGBLED-MX-1U-RGB, K29 KEYSWITCH-RGBLED-MX-1U-RGB, K3 KEYSWITCH-RGBLED-MX-1U-RGB, K30 KEYSWITCH-RGBLED-MX-1U-RGB, K31 KEYSWITCH-RGBLED-MX-1U-RGB, K32 KEYSWITCH-RGBLED-MX-1U-RGB, K33 KEYSWITCH-RGBLED-MX-1U-RGB, K34 KEYSWITCH-RGBLED-MX-1U-RGB, K35 KEYSWITCH-RGBLED-MX-1U-RGB, K36 KEYSWITCH-RGBLED-MX-1U-RGB, K37 KEYSWITCH-RGBLED-MX-1U-RGB, K38 KEYSWITCH-RGBLED-MX-1U-RGB, K39 KEYSWITCH-RGBLED-MX-1U-RGB, K4 KEYSWITCH-RGBLED-MX-1U-RGB, K40 KEYSWITCH-RGBLED-MX-1U-RGB, K41 KEYSWITCH-RGBLED-MX-1U-RGB, K42 KEYSWITCH-RGBLED-MX-1U-RGB, K5 KEYSWITCH-RGBLED-MX-1U-RGB, K6 KEYSWITCH-RGBLED-MX-1U-RGB, K7 KEYSWITCH-RGBLED-MX-1U-RGB, K8 KEYSWITCH-RGBLED-MX-1U-RGB, K9 KEYSWITCH-RGBLED-MX-1U-RGB

Commit message: updated sch and brd files
Parts:
- removed D15, D16, D17, D18, D19, D20, D21, D22, D23, D24, D25, D26, D28, D29, D30, D31, D32, D33, D34, D35, D36, D37, D38, D39: (no value), Components:DIODE-DFN0603-2
- removed K17, K18, K19, K20, K21, K22, K23, K24, K25, K26, K27, K28, K29, K30, K31, K32, K33, K34, K35, K36, K37, K38, K39, K40, K41, K42: KEYSWITCH-RGBLED-MX-1U-RGB, Keyboard:KEYSWITCH-RGBLED-MX-1U-RGB
- K1, K10, K11, K12, K13, K14, K15, K16, K2, K3, K4, K5, K6, K7, K8, K9: value KEYSWITCH-RGBLED-MX-1U-RGB -> KEYSWITCH-LEDTHTHOLE-MXHS-1U-LEDTHTHOLE; device Keyboard:KEYSWITCH-RGBLED-MX-1U-RGB -> Keyboard:KEYSWITCH-LEDTHTHOLE-MXHS-1U-LEDTHTHOLE
Connections:
- removed net COL10: K11.P0, K25.P0, K39.P0
- removed net COL11: K12.P0, K26.P0, K40.P0
- removed net COL12: K13.P0, K27.P0, K41.P0
- removed net COL13: K14.P0, K28.P0, K42.P0
- removed net COL2: K17.P0, K3.P0, K31.P0
- removed net COL3: K18.P0, K32.P0, K4.P0
- removed net COL4: K19.P0, K33.P0, K5.P0
- removed net COL5: K20.P0, K34.P0, K6.P0
- removed net COL6: K21.P0, K35.P0, K7.P0
- removed net COL7: K22.P0, K36.P0, K8.P0
- removed net COL8: K23.P0, K37.P0, K9.P0
- removed net COL9: K10.P0, K24.P0, K38.P0
- removed net N$19: D14.C, D15.A, K16.P1
- removed net N$25: D26.C, K28.P1
- removed net N$26: D25.C, D26.A, K27.P1
- removed net N$27: D24.C, D25.A, K26.P1
- removed net N$28: D23.C, D24.A, K25.P1
- removed net N$29: D22.C, D23.A, K24.P1
- removed net N$30: D21.C, D22.A, K23.P1
- removed net N$31: D20.C, D21.A, K22.P1
- removed net N$32: D19.C, D20.A, K21.P1
- removed net N$33: D18.C, D19.A, K20.P1
- removed net N$34: D17.C, D18.A, K19.P1
- removed net N$35: D16.C, D17.A, K18.P1
- removed net N$36: D15.C, D16.A, K17.P1
- removed net N$37: D27.C, D28.A, K30.P1
- removed net N$38: D39.C, K42.P1
- removed net N$39: D38.C, D39.A, K41.P1
- removed net N$40: D37.C, D38.A, K40.P1
- removed net N$41: D36.C, D37.A, K39.P1
- removed net N$42: D35.C, D36.A, K38.P1
- removed net N$43: D34.C, D35.A, K37.P1
- removed net N$44: D33.C, D34.A, K36.P1
- removed net N$45: D32.C, D33.A, K35.P1
- removed net N$46: D31.C, D32.A, K34.P1
- removed net N$47: D30.C, D31.A, K33.P1
- removed net N$48: D29.C, D30.A, K32.P1
- removed net N$49: D28.C, D29.A, K31.P1
- net COL0: now also K16.P0; no longer K29.P0
- net COL1: no longer K16.P0, K2.P0, K30.P0
- net ROW2: now also K16.P1; no longer K29.P1
